Commit message: reformatted code

File: usv_sim/xacro/mr1_hull.xacro (robot description, xacro)
@@ -38,13 +38,13 @@
           </inertial>
           <buoyancy>
-        <compensation>${middle_water_displaced_mass/middle_body_mass}</compensation>
-        <origin xyz="${0.35*scale} ${0.44*scale} ${-0.15*scale}"/>
-        <limit radius="0.1"/>
-        <damping rpy="20 20 20" xyz="20 40 50"/>
+            <compensation>${middle_water_displaced_mass/middle_body_mass}</compensation>
+            <origin xyz="${0.35*scale} ${0.44*scale} ${-0.15*scale}"/>
+            <limit radius="0.1"/>
+            <damping rpy="20 20 20" xyz="20 40 50"/>
             <windVelocity>${windType}</windVelocity>
-        <frontal_area>0.0</frontal_area>
-        <lateral_area>0.06</lateral_area>
-        <lateral_length>1.2</lateral_length>
-          <waterVelocity>${waterType}</waterVelocity>
+            <frontal_area>0.0</frontal_area>
+            <lateral_area>0.06</lateral_area>
+            <lateral_length>1.2</lateral_length>
+            <waterVelocity>${waterType}</waterVelocity>
           </buoyancy>
       </link>
@@ -52,5 +52,5 @@
         <parent link="${parentLink}"/>
         <child link="${name}_center_l_link"/>
-        <origin rpy="0 0 ${ninety_degrees}" xyz="0 0 0"/>
+        <origin rpy="0 0 ${ninety_degrees}" xyz="0 0 -0.2"/>
       </joint>
       <link name="${name}_center_r_link">
