Commit message: fixed indentation

File: usv_sim/xacro/sailboat.xacro (robot description, xacro)
@@ -108,5 +108,6 @@
 		  <forward>1 0 0</forward>
 		  <upward>0 1 0</upward>
-		  <link_name>keel</link_name>
+	        <limit effort="100" velocity="70" lower="-${PI}" upper="${PI}" />
+	  <link_name>keel</link_name>
 		  <fluidVelocity>${waterType}</fluidVelocity>
     </plugin>
