Commit message: added collision and inertia

File: usv_sim/xacro/mr1_base_frame.xacro (robot description, xacro)
@@ -1,4 +1,4 @@
 <?xml version="1.0"?>
-<robot xmlns:xacro="http://www.ros.org/wiki/xacro" name="mr1_base_frame">
+<xacro xmlns:xacro="http://www.ros.org/wiki/xacro" name="mr1_base_frame">
   <xacro:property name="beam_length" value="0.6" />
   <xacro:property name="beam_radius" value="0.055" />
@@ -13,4 +13,14 @@
       <origin rpy="0 0 0 " xyz="0 0 0"/>
     </visual>
+    <collision>
+      <geometry>
+        <box size="${base_cube_length} ${base_cube_length} ${base_cube_length}"/>
+      </geometry>
+      <origin rpy="0 0 0 " xyz="0 0 0"/>
+    </collision>
+    <inertial>
+      <mass value="1"/>
+      <inertia ixx="0.01" ixy="0.0" ixz="0.0" iyy="0.01" iyz="0.0" izz="0.01"/>
+    </inertial>
   </link>
   <link name="right_beam">
@@ -22,4 +32,15 @@
       <origin rpy="0 ${ninety_degrees} 0" xyz="0 0 0"/>
     </visual>
+    <collision>
+      <geometry>
+        <cylinder radius="${beam_radius}" length="${beam_length}"/>
+      </geometry>
+      <!-- rotate beam 90 degrees -->
+      <origin rpy="0 ${ninety_degrees} 0" xyz="0 0 0"/>
+    </collision>
+    <inertial>
+      <mass value="1"/>
+      <inertia ixx="0.01" ixy="0.0" ixz="0.0" iyy="0.01" iyz="0.0" izz="0.01"/>
+    </inertial>
   </link>
   <joint name="base_to_right_leg" type="fixed">
@@ -35,4 +56,14 @@
       <origin rpy="0 ${ninety_degrees} 0" xyz="0 0 0"/>
     </visual>
+    <collision>
+      <geometry>
+        <cylinder radius="${beam_radius}" length="${beam_length}"/>
+      </geometry>
+      <origin rpy="0 ${ninety_degrees} 0" xyz="0 0 0"/>
+    </collision>
+    <inertial>
+      <mass value="1"/>
+      <inertia ixx="0.01" ixy="0.0" ixz="0.0" iyy="0.01" iyz="0.0" izz="0.01"/>
+    </inertial>
   </link>
   <joint name="base_to_left_beam" type="fixed">
@@ -49,4 +80,15 @@
       <origin rpy="0 0 0" xyz="0 0 ${-beam_to_hull_length/2}"/>
     </visual>
+    <collision>
+      <geometry>
+        <cylinder radius="${beam_radius}" length="${beam_to_hull_length}"/>
+      </geometry>
+      <!--origin z offset = length/2 -->
+      <origin rpy="0 0 0" xyz="0 0 ${-beam_to_hull_length/2}"/>
+    </collision>
+    <inertial>
+      <mass value="1"/>
+      <inertia ixx="0.01" ixy="0.0" ixz="0.0" iyy="0.01" iyz="0.0" izz="0.01"/>
+    </inertial>
   </link>
   <joint name="left_beam_to_attachment" type="fixed">
@@ -64,4 +106,15 @@
       <origin rpy="0 0 0" xyz="0 0 ${-beam_to_hull_length/2}"/>
     </visual>
+    <collision>
+      <geometry>
+        <cylinder radius="${beam_radius}" length="${beam_to_hull_length}"/>
+      </geometry>
+      <!--origin z offset = length/2 -->
+      <origin rpy="0 0 0" xyz="0 0 ${-beam_to_hull_length/2}"/>
+    </collision>
+    <inertial>
+      <mass value="1"/>
+      <inertia ixx="0.01" ixy="0.0" ixz="0.0" iyy="0.01" iyz="0.0" izz="0.01"/>
+    </inertial>
   </link>
   <joint name="right_beam_to_attachment" type="fixed">
@@ -71,3 +124,3 @@
     <origin xyz="0.25 0 0"/>
   </joint>
-</robot>
+</xacro>

Commit message: renamed 'base_link' to 'base_cube'

File: usv_sim/xacro/mr1_base_frame.xacro (robot description, xacro)
@@ -6,5 +6,5 @@
   <xacro:property name="beam_to_hull_length" value="0.1778" />
   <xacro:property name="ninety_degrees" value="1.57075" />
-  <link name="base_link">
+  <link name="base_cube">
     <visual>
       <geometry>
@@ -45,5 +45,5 @@
   </link>
   <joint name="base_to_right_leg" type="fixed">
-    <parent link="base_link"/>
+    <parent link="base_cube"/>
     <child link="right_beam"/>
     <origin xyz="${(beam_length/2)+(base_cube_length/2)} 0 0"/>
@@ -68,5 +68,5 @@
   </link>
   <joint name="base_to_left_beam" type="fixed">
-    <parent link="base_link"/>
+    <parent link="base_cube"/>
     <child link="left_beam"/>
     <origin xyz="${-((beam_length/2)+(base_cube_length/2))} 0 0"/>

Commit message: added rear beam and rudder macro

File: usv_sim/xacro/mr1_base_frame.xacro (robot description, xacro)
@@ -4,5 +4,5 @@
   <xacro:property name="beam_radius" value="0.055" />
   <xacro:property name="base_cube_length" value="0.12" />
-  <xacro:property name="beam_to_hull_length" value="0.1778" />
+  <xacro:property name="beam_to_hull_length" value="0.0889" />
   <xacro:property name="ninety_degrees" value="1.57075" />
   <link name="base_cube">
@@ -24,4 +24,27 @@
     </inertial>
   </link>
+  <link name="rear_beam">
+    <visual>
+      <geometry>
+        <cylinder radius="${beam_radius}" length="${beam_length}"/>
+      </geometry>
+      <origin rpy="${ninety_degrees} 0 0" xyz="0 0 0"/>
+    </visual>
+    <collision>
+      <geometry>
+        <cylinder radius="${beam_radius}" length="${beam_length}"/>
+      </geometry>
+      <origin rpy="${ninety_degrees} 0 0" xyz="0 0 0"/>
+    </collision>
+    <inertial>
+      <mass value="1"/>
+      <inertia ixx="0.01" ixy="0.0" ixz="0.0" iyy="0.01" iyz="0.0" izz="0.01"/>
+    </inertial>
+  </link>
+  <joint name="base_to_rear_beam" type="fixed">
+    <parent link="base_cube"/>
+    <child link="rear_beam"/>
+    <origin xyz="0 ${-(beam_length/2)+(base_cube_length/2)} 0"/>
+  </joint>
   <link name="right_beam">
     <visual>
@@ -124,3 +147,64 @@
     <origin xyz="0.25 0 0"/>
   </joint>
+ <link name="rudder_attachment">
+    <visual>
+      <geometry>
+        <cylinder radius="${beam_radius}" length="${beam_to_hull_length}"/>
+      </geometry>
+      <!--origin z offset = length/2 -->
+      <origin rpy="0 0 0" xyz="0 0 ${-beam_to_hull_length/2}"/>
+    </visual>
+    <collision>
+      <geometry>
+        <cylinder radius="${beam_radius}" length="${beam_to_hull_length}"/>
+      </geometry>
+      <!--origin z offset = length/2 -->
+      <origin rpy="0 0 0" xyz="0 0 ${-beam_to_hull_length/2}"/>
+    </collision>
+    <inertial>
+      <mass value="1"/>
+      <inertia ixx="0.01" ixy="0.0" ixz="0.0" iyy="0.01" iyz="0.0" izz="0.01"/>
+    </inertial>
+  </link>
+  <joint name="rear_beam_to_attachment" type="fixed">
+    <parent link="rear_beam"/>
+    <child link="rudder_attachment"/>
+    <!--origin x offset = beam_length/2 -radius -->
+    <origin xyz="0 -0.25 0"/>
+  </joint>
+  <!-- Rudder link -->
+    <xacro:macro name="rudder_xacro">
+        <link name="rudder">
+            <inertial>
+                <mass value="1" />
+                <inertia
+                  ixx="0.05"
+                  ixy="0.0"
+                  iyy="0.05"
+                  ixz="0.0"
+                  iyz="0.0"
+                  izz="0.005"/>
+            </inertial>
+            <collision name="collision">
+                <geometry>
+                  <box size="${0.2*scale} ${0.02*scale} ${0.3*scale}" />
+                </geometry>
+                <origin rpy="0 0 0" xyz="${-0.1*scale} 0 0"/>
+            </collision>
+            <visual name="visual">
+                <geometry>
+                  <mesh filename="package://usv_sim/meshes/simpleHull3/box.dae" scale="${0.2*scale} ${0.02*scale} ${0.3*scale}"/>
+                </geometry>
+                <origin rpy="0 0 0" xyz="${-0.1*scale} 0 0"/>
+            </visual>
+        </link>
+        <joint name="rudder_joint" type="revolute">
+            <parent link="rudder_attachment"/>
+            <child link="rudder"/>
+            <origin rpy="0 0 0" xyz="0 0 ${-1.5*scale}"/>
+            <dynamics damping="1.0"/>
+            <axis xyz="0 0 1"/>
+            <limit effort="100" velocity="5" lower="-${PI/2}" upper="${PI/2}" />
+        </joint>
+    </xacro:macro>
 </xacro>

Commit message: moved rudder back and up

File: usv_sim/xacro/mr1_base_frame.xacro (robot description, xacro)
@@ -190,5 +190,5 @@
                   <box size="${0.2*scale} ${0.02*scale} ${0.3*scale}" />
                 </geometry>
-                <origin rpy="0 0 0" xyz="${-0.1*scale} 0 0"/>
+                <origin rpy="0 0 0" xyz="${-0.2*scale} 0 0"/>
             </collision>
             <visual name="visual">
@@ -196,5 +196,5 @@
                   <mesh filename="package://usv_sim/meshes/simpleHull3/box.dae" scale="${0.2*scale} ${0.02*scale} ${0.3*scale}"/>
                 </geometry>
-                <origin rpy="0 0 0" xyz="${-0.1*scale} 0 0"/>
+                <origin rpy="0 0 0" xyz="${-0.2*scale} 0 0"/>
             </visual>
         </link>
@@ -202,5 +202,5 @@
             <parent link="rudder_attachment"/>
             <child link="rudder"/>
-            <origin rpy="0 0 0" xyz="0 0 ${-1.5*scale}"/>
+            <origin rpy="0 0 ${ninety_degrees}" xyz="0 0 ${-1.2*scale}"/>
             <dynamics damping="1.0"/>
             <axis xyz="0 0 1"/>

Commit message: modified to work with new hull, modified rudder joit

File: usv_sim/xacro/mr1_base_frame.xacro (robot description, xacro)
@@ -4,5 +4,5 @@
   <xacro:property name="beam_radius" value="0.055" />
   <xacro:property name="base_cube_length" value="0.12" />
-  <xacro:property name="beam_to_hull_length" value="0.0889" />
+  <xacro:property name="beam_to_hull_length" value="0.254" />
   <xacro:property name="ninety_degrees" value="1.57075" />
   <link name="base_cube">
@@ -11,5 +11,5 @@
         <box size="${base_cube_length} ${base_cube_length} ${base_cube_length}"/>
       </geometry>
-      <origin rpy="0 0 0 " xyz="0 0 0"/>
+      <origin rpy="0 0 0" xyz="0 0 0"/>
     </visual>
     <collision>
@@ -17,5 +17,5 @@
         <box size="${base_cube_length} ${base_cube_length} ${base_cube_length}"/>
       </geometry>
-      <origin rpy="0 0 0 " xyz="0 0 0"/>
+      <origin rpy="0 0 0" xyz="0 0 0"/>
     </collision>
     <inertial>
@@ -188,5 +188,5 @@
             <collision name="collision">
                 <geometry>
-                  <box size="${0.2*scale} ${0.02*scale} ${0.3*scale}" />
+                  <box size="${0.2*scale} ${0.02*scale} ${0.6*scale}" />
                 </geometry>
                 <origin rpy="0 0 0" xyz="${-0.2*scale} 0 0"/>
@@ -194,5 +194,5 @@
             <visual name="visual">
                 <geometry>
-                  <mesh filename="package://usv_sim/meshes/simpleHull3/box.dae" scale="${0.2*scale} ${0.02*scale} ${0.3*scale}"/>
+                  <mesh filename="package://usv_sim/meshes/simpleHull3/box.dae" scale="${0.2*scale} ${0.02*scale} ${0.6*scale}"/>
                 </geometry>
                 <origin rpy="0 0 0" xyz="${-0.2*scale} 0 0"/>
@@ -202,8 +202,9 @@
             <parent link="rudder_attachment"/>
             <child link="rudder"/>
-            <origin rpy="0 0 ${ninety_degrees}" xyz="0 0 ${-1.2*scale}"/>
+            <origin rpy="0 0 ${ninety_degrees}" xyz="0 0 ${-0.6*scale}"/>
+<!--            <origin rpy="0 0 ${ninety_degrees" xyz="0 0 ${-0.6*scale}"/-->
             <dynamics damping="1.0"/>
             <axis xyz="0 0 1"/>
-            <limit effort="100" velocity="5" lower="-${PI/2}" upper="${PI/2}" />
+            <limit effort="100" velocity="5" lower="-${PI/4}" upper="${PI/4}" />
         </joint>
     </xacro:macro>
