Commit message: flipped join origin y value for correct hull shape

File: usv_sim/xacro/mr1_right_hull.xacro (robot description, xacro)
@@ -81,5 +81,5 @@
         <parent link="center_r_link"/>
         <child link="back_r_link"/>
-        <origin rpy="0 0 0" xyz="${-0.5*scale} ${0.39*scale} 0"/>
+        <origin rpy="0 0 0" xyz="${-0.5*scale} ${-0.39*scale} 0"/>
 	<limit effort="50" velocity="5" lower="0" upper="0" />
             <dynamics damping="1.0"/>
@@ -119,5 +119,5 @@
         <parent link="center_r_link"/>
         <child link="front_r_link"/>
-        <origin rpy="0 0 0" xyz="${1.3*scale} ${0.2*scale} 0"/>
+        <origin rpy="0 0 0" xyz="${1.3*scale} ${-0.2*scale} 0"/>
 	<limit effort="50" velocity="5" lower="0" upper="0" />
             <dynamics damping="1.0"/>

Commit message: removed yaw adjustment from buoyancy

File: usv_sim/xacro/mr1_right_hull.xacro (robot description, xacro)
@@ -25,5 +25,5 @@
     <buoyancy>
       <compensation>${middle_water_displaced_mass/middle_body_mass}</compensation>
-      <origin xyz="${-1.2619*scale} ${-1.71630000002334E-07*scale} ${-0.038115*scale}" rpy="0 0 ${-ninety_degrees}"/>
+      <origin xyz="${-1.2619*scale} ${-1.71630000002334E-07*scale} ${-0.038115*scale}" rpy="0 0 0"/>
       <limit radius="0.1"/>
       <damping rpy="20 20 20" xyz="20 40 50"/>
@@ -59,5 +59,5 @@
     <buoyancy>
       <compensation>${back_water_displaced_mass/back_body_mass}</compensation>
-      <origin xyz="${-0.55395*scale} ${-9.49220000000195E-06*scale} ${-0.031774*scale}" rpy="0 0 ${-ninety_degrees}"/>
+      <origin xyz="${-0.55395*scale} ${-9.49220000000195E-06*scale} ${-0.031774*scale}" rpy="0 0 0"/>
       <limit radius="0.1"/>
       <damping rpy="20 20 20" xyz="20 40 50"/>
@@ -101,5 +101,5 @@
     <buoyancy>
       <compensation>${front_water_displaced_mass/front_body_mass}</compensation>
-      <origin xyz="${-1.9778*scale} ${4.47239999998292E-07*scale} ${-0.027892*scale}" rpy="0 0 ${-ninety_degrees}" />
+      <origin xyz="${-1.9778*scale} ${4.47239999998292E-07*scale} ${-0.027892*scale}" rpy="0 0 0" />
       <limit radius="0.1"/>
       <damping rpy="20 20 20" xyz="20 40 50"/>
