Commit message: removed xacro properties (moved to mr1.xacro)

File: usv_sim/xacro/mr1_left_hull.xacro (robot description, xacro)
@@ -1,21 +1,4 @@
 <?xml version="1.0"?>
 <xacro xmlns:xacro="http://www.ros.org/wiki/xacro">
-    <xacro:property name="PI" value="3.1415926535897931"/>
-    <!-- Body properties -->
-    <xacro:property name="front_body_mass" value="5"/>
-    <xacro:property name="back_body_mass" value="5"/>
-    <xacro:property name="middle_body_mass" value="5"/>
-    <xacro:property name="rear_body_mass" value="5"/>
-    <xacro:property name="front_body_mass" value="2"/>
-    <xacro:property name="back_water_displaced_mass" value="40"/>
-    <xacro:property name="middle_water_displaced_mass" value="40"/>
-    <xacro:property name="front_water_displaced_mass" value="25"/>
-    <xacro:property name="scale" value="0.3"/>
-    <xacro:property name="bl1" value=".1" />
-    <xacro:property name="bl2" value=".1" />
-    <xacro:arg name="windType" default="global" />
-    <xacro:arg name="waterType" default="global" />
-    <xacro:property name="windType" value="$(arg windType)" />
-    <xacro:property name="waterType" value="$(arg waterType)" />
     <link name="base_link">
         <visual>

File: usv_sim/xacro/mr1_right_hull.xacro (robot description, xacro)
@@ -1,21 +1,4 @@
 <?xml version="1.0"?>
 <xacro xmlns:xacro="http://www.ros.org/wiki/xacro">
-    <xacro:property name="PI" value="3.1415926535897931"/>
-    <!-- Body properties -->
-    <xacro:property name="front_body_mass" value="5"/>
-    <xacro:property name="back_body_mass" value="5"/>
-    <xacro:property name="middle_body_mass" value="5"/>
-    <xacro:property name="rear_body_mass" value="5"/>
-    <xacro:property name="front_body_mass" value="2"/>
-    <xacro:property name="back_water_displaced_mass" value="40"/>
-    <xacro:property name="middle_water_displaced_mass" value="40"/>
-    <xacro:property name="front_water_displaced_mass" value="25"/>
-    <xacro:property name="scale" value="0.3"/>
-    <xacro:property name="bl1" value=".1" />
-    <xacro:property name="bl2" value=".1" />
-    <xacro:arg name="windType" default="global" />
-    <xacro:arg name="waterType" default="global" />
-    <xacro:property name="windType" value="$(arg windType)" />
-    <xacro:property name="waterType" value="$(arg waterType)" />
     <link name="center_r_link">
         <visual>

Commit message: switched to hull size and meshes exported from solidworks

File: usv_sim/xacro/mr1_left_hull.xacro (robot description, xacro)
@@ -1,109 +1,121 @@
 <?xml version="1.0"?>
-<xacro xmlns:xacro="http://www.ros.org/wiki/xacro">
-    <link name="base_link">
-        <visual>
-          <origin rpy="0 0 0" xyz="0 0 0"/>
-          <geometry>
-            <mesh filename="package://usv_sim/meshes/simpleHull3/base_link.dae" scale="${scale} ${scale} ${scale}"/>
-          </geometry>
-        </visual>
-        <collision>
-          <origin rpy="0 0 0" xyz="0 0 0"/>
-          <geometry>
-            <mesh filename="package://usv_sim/meshes/simpleHull3/base_link.dae" scale="${scale} ${scale} ${scale}"/>
-          </geometry>
-        </collision>
-        <inertial>
-            <origin rpy="0 0 0" xyz="${0.35*scale} ${0.44*scale} ${-0.2*scale}"/>
-          <mass value="${middle_body_mass}"/>
-          <inertia ixx="0.1" ixy="0.0" ixz="0.0" iyy="1.4" iyz="0.0" izz="1.4"/>
-        </inertial>
-        <buoyancy>
-			<compensation>${middle_water_displaced_mass/middle_body_mass}</compensation>
-			<origin xyz="${0.35*scale} ${0.44*scale} ${-0.15*scale}"/>
-			<limit radius="0.1"/>
-			<damping rpy="20 20 20" xyz="20 40 50"/>
-         	<windVelocity>${windType}</windVelocity>
-			<frontal_area>0.0</frontal_area>
-			<lateral_area>0.06</lateral_area>
-			<lateral_length>1.2</lateral_length>
-	  		<waterVelocity>${waterType}</waterVelocity>
-        </buoyancy>
-    </link>
-    <link name="back_l_link">
-        <visual>
-          <origin rpy="0 0 0"  xyz="0 0 0"/>
-          <geometry>
-           	<mesh filename="package://usv_sim/meshes/simpleHull3/backLeft.dae" scale="${scale} ${scale} ${scale}"/>
-          </geometry>
-        </visual>
-        <collision>
-          <origin rpy="0 0 0"  xyz="0 0 0"/>
-          <geometry>
-           	<mesh filename="package://usv_sim/meshes/simpleHull3/backLeft.dae" scale="${scale} ${scale} ${scale}"/>
-          </geometry>
-        </collision>
-        <inertial>
-            <origin rpy="0 0 0" xyz="${-0.6*scale} 0 ${-0.2*scale}"/>
-          <mass value="${back_body_mass}"/>
-          <inertia ixx="0.1" ixy="0.0" ixz="0.0" iyy="1.4" iyz="0.0" izz="1.4"/>
-        </inertial>
-        <buoyancy>
-			<compensation>${back_water_displaced_mass/back_body_mass}</compensation>
-			<origin xyz="${-0.6*scale} 0 ${-0.15*scale}"/>
-			<limit radius="0.1"/>
-			<damping rpy="20 20 20" xyz="20 40 50"/>
-			<windVelocity>${windType}</windVelocity>
-			<frontal_area>0.04</frontal_area>
-			<lateral_area>0.06</lateral_area>
-			<lateral_length>1.2</lateral_length>
-	  		<waterVelocity>${waterType}</waterVelocity>
-        </buoyancy>
-    </link>
-    <joint name="back_l_joint" type="revolute">
-        <parent link="base_link"/>
-        <child link="back_l_link"/>
-        <origin rpy="0 0 0" xyz="${-0.5*scale} ${0.39*scale} 0"/>
-	<limit effort="50" velocity="5" lower="0" upper="0" />
-            <dynamics damping="1.0"/>
-            <axis xyz="1 0 0"/>
-    </joint>
-    <link name="front_l_link">
-    	<visual>
-    	<origin rpy="0 0 0"  xyz="0 0 0"/>
-          <geometry>
-           	<mesh filename="package://usv_sim/meshes/simpleHull3/frontLeft.dae" scale="${scale} ${scale} ${scale}"/>
-          </geometry>
-    	</visual>
-        <collision>
-          <origin rpy="0 0 0"  xyz="0 0 0"/>
-          <geometry>
-           	<mesh filename="package://usv_sim/meshes/simpleHull3/frontLeft.dae" scale="${scale} ${scale} ${scale}"/>
-          </geometry>
-        </collision>
-        <inertial>
-            <origin rpy="0 0 0" xyz="${0.4*scale} 0 ${-0.1*scale}"/>
-          <mass value="${front_body_mass}"/>
-          <inertia ixx="0.1" ixy="0.0" ixz="0.0" iyy="1.4" iyz="0.0" izz="1.4"/>
-        </inertial>
-        <buoyancy>
-          	<compensation>${front_water_displaced_mass/front_body_mass}</compensation>
-          	<origin xyz="${0.4*scale} 0 ${-0.05*scale}"/>
-          	<limit radius="0.1"/>
-          	<damping rpy="20 20 20" xyz="20 40 50"/>
-          	<windVelocity>${windType}</windVelocity>
-			<frontal_area>0.04</frontal_area>
-			<lateral_area>0.06</lateral_area>
-			<lateral_length>1.2</lateral_length>
-	  		<waterVelocity>${waterType}</waterVelocity>
-        </buoyancy>
-    </link>
-    <joint name="front_l_joint" type="revolute">
-        <parent link="base_link"/>
-        <child link="front_l_link"/>
-        <origin rpy="0 0 0" xyz="${1.3*scale} ${0.2*scale} 0"/>
-	<limit effort="50" velocity="5" lower="0" upper="0" />
-            <dynamics damping="1.0"/>
-            <axis xyz="1 0 0"/>
-    </joint>
+<xacro xmlns:xacro="http://www.ros.org/wiki/xacro" name="left_hull">
+  <!--MR1 BASE LINK-->
+  <link name="base_link">
+    <inertial>
+      <origin xyz="${-1.2619*scale} ${-1.71630000002334E-07*scale} ${-0.038115*scale}" rpy="0 0 0" />
+      <mass value="${3.333*scale}" />
+      <inertia ixx="0.61191" ixy="6.46809999999998E-05" ixz="0.0040806" iyy="3.5097" iyz="1.36870000000023E-05" izz="3.5471" />
+    </inertial>
+    <visual>
+      <origin xyz="0 0 0" rpy="1.5707963267949 0 0" />
+      <geometry>
+        <mesh filename="package://usv_sim/meshes/Hull-Middle.STL" />
+      </geometry>
+      <material name="">
+        <color rgba="0.75294 0.75294 0.75294 1" />
+      </material>
+    </visual>
+    <collision>
+      <origin xyz="0 0 0" rpy="1.5707963267949 0 0" />
+      <geometry>
+        <mesh filename="package://usv_sim/meshes/Hull-Middle.STL" />
+      </geometry>
+    </collision>
+    <buoyancy>
+      <compensation>${middle_water_displaced_mass/middle_body_mass}</compensation>
+      <origin xyz="${-1.2619*scale} ${-1.71630000002334E-07*scale} ${-0.038115*scale}" rpy="0 0 0"/>
+      <limit radius="0.1"/>
+      <damping rpy="20 20 20" xyz="20 40 50"/>
+      <windVelocity>${windType}</windVelocity>
+      <frontal_area>0.0</frontal_area>
+      <lateral_area>0.06</lateral_area>
+      <lateral_length>1.2</lateral_length>
+      <waterVelocity>${waterType}</waterVelocity>
+    </buoyancy>
+  </link>
+  <!--MR1 BACK LINK-->
+  <link name="back_l_link">
+    <inertial>
+      <origin xyz="${-0.55395*scale} ${-9.49220000000195E-06*scale} ${-0.031774*scale}" rpy="0 0 0" />
+      <mass value="${3.333*scale}" />
+      <inertia ixx="0.22991" ixy="-2.0064999999998E-05" ixz="-0.032423" iyy="1.3348" iyz="-4.95610000000025E-05" izz="1.2943" />
+    </inertial>
+    <visual>
+      <origin xyz="0 0 0" rpy="1.5707963267949 0 0" />
+      <geometry>
+        <mesh filename="package://usv_sim/meshes/Hull-Back.STL" />
+      </geometry>
+      <material name="">
+        <color rgba="0.75294 0.75294 0.75294 1" />
+      </material>
+    </visual>
+    <collision>
+      <origin xyz="0 0 0" rpy="1.5707963267949 0 0" />
+      <geometry>
+        <mesh filename="package://usv_sim/meshes/Hull-Back.STL" />
+      </geometry>
+    </collision>
+    <buoyancy>
+      <compensation>${back_water_displaced_mass/back_body_mass}</compensation>
+      <origin xyz="${-0.55395*scale} ${-9.49220000000195E-06*scale} ${-0.031774*scale}"/>
+      <limit radius="0.1"/>
+      <damping rpy="20 20 20" xyz="20 40 50"/>
+      <windVelocity>${windType}</windVelocity>
+      <frontal_area>0.04</frontal_area>
+      <lateral_area>0.06</lateral_area>
+      <lateral_length>1.2</lateral_length>
+      <waterVelocity>${waterType}</waterVelocity>
+    </buoyancy>
+  </link>
+  <joint name="back_l_joint" type="revolute">
+    <parent link="base_link"/>
+    <child link="back_l_link"/>
+    <origin rpy="0 0 0" xyz="0 0 0"/>
+    <limit effort="50" velocity="5" lower="0" upper="0" />
+    <dynamics damping="1.0"/>
+    <axis xyz="1 0 0"/>
+  </joint>
+  <!--MR1 FRONT LINK-->
+  <link name="front_l_link">
+    <inertial>
+      <origin xyz="${-1.9778*scale} ${4.47239999998292E-07*scale} ${-0.027892*scale}" rpy="0 0 0" />
+      <mass value="${3.333*scale}" />
+      <inertia ixx="0.1729" ixy="1.57389999997978E-07" ixz="0.033027" iyy="1.1311" iyz="3.95489999997434E-07" izz="1.0892" />
+    </inertial>
+    <visual>
+      <origin xyz="0 0 0" rpy="1.5707963267949 0 0" />
+      <geometry>
+        <mesh filename="package://usv_sim/meshes/Hull-Front.STL" />
+      </geometry>
+      <material name="">
+        <color rgba="0.75294 0.75294 0.75294 1" />
+      </material>
+    </visual>
+    <collision>
+      <origin xyz="0 0 0" rpy="1.5707963267949 0 0" />
+      <geometry>
+        <mesh filename="package://usv_sim/meshes/Hull-Front.STL" />
+      </geometry>
+    </collision>
+    <buoyancy>
+      <compensation>${front_water_displaced_mass/front_body_mass}</compensation>
+      <origin xyz="${-1.9778*scale} ${4.47239999998292E-07*scale} ${-0.027892*scale}" rpy="0 0 0" />
+      <limit radius="0.1"/>
+      <damping rpy="20 20 20" xyz="20 40 50"/>
+      <windVelocity>${windType}</windVelocity>
+      <frontal_area>0.04</frontal_area>
+      <lateral_area>0.06</lateral_area>
+      <lateral_length>1.2</lateral_length>
+      <waterVelocity>${waterType}</waterVelocity>
+    </buoyancy>
+  </link>
+  <joint name="front_l_joint" type="revolute">
+    <parent link="base_link"/>
+    <child link="front_l_link"/>
+    <origin rpy="0 0 0" xyz="0 0 0"/>
+    <limit effort="50" velocity="5" lower="0" upper="0" />
+    <dynamics damping="1.0"/>
+    <axis xyz="1 0 0"/>
+  </joint>
 </xacro>

File: usv_sim/xacro/mr1_right_hull.xacro (robot description, xacro)
@@ -1,109 +1,121 @@
 <?xml version="1.0"?>
-<xacro xmlns:xacro="http://www.ros.org/wiki/xacro">
-    <link name="center_r_link">
-        <visual>
-          <origin rpy="0 0 0" xyz="0 0 0"/>
-          <geometry>
-            <mesh filename="package://usv_sim/meshes/simpleHull3/centerRight.dae" scale="${scale} ${scale} ${scale}"/>
-          </geometry>
-        </visual>
-        <collision>
-          <origin rpy="0 0 0" xyz="0 0 0"/>
-          <geometry>
-            <mesh filename="package://usv_sim/meshes/simpleHull3/centerRight.dae" scale="${scale} ${scale} ${scale}"/>
-          </geometry>
-        </collision>
-        <inertial>
-            <origin rpy="0 0 0" xyz="${0.35*scale} ${0.44*scale} ${-0.2*scale}"/>
-          <mass value="${middle_body_mass}"/>
-          <inertia ixx="0.1" ixy="0.0" ixz="0.0" iyy="1.4" iyz="0.0" izz="1.4"/>
-        </inertial>
-        <buoyancy>
-			<compensation>${middle_water_displaced_mass/middle_body_mass}</compensation>
-			<origin xyz="${0.35*scale} ${0.44*scale} ${-0.15*scale}"/>
-			<limit radius="0.1"/>
-			<damping rpy="20 20 20" xyz="20 40 50"/>
-         	<windVelocity>${windType}</windVelocity>
-			<frontal_area>0.0</frontal_area>
-			<lateral_area>0.06</lateral_area>
-			<lateral_length>1.2</lateral_length>
-	  		<waterVelocity>${waterType}</waterVelocity>
-        </buoyancy>
-    </link>
-    <link name="back_r_link">
-        <visual>
-          <origin rpy="0 0 0"  xyz="0 0 0"/>
-          <geometry>
-           	<mesh filename="package://usv_sim/meshes/simpleHull3/backRight.dae" scale="${scale} ${scale} ${scale}"/>
-          </geometry>
-        </visual>
-        <collision>
-          <origin rpy="0 0 0"  xyz="0 0 0"/>
-          <geometry>
-           	<mesh filename="package://usv_sim/meshes/simpleHull3/backRight.dae" scale="${scale} ${scale} ${scale}"/>
-          </geometry>
-        </collision>
-        <inertial>
-            <origin rpy="0 0 0" xyz="${-0.6*scale} 0 ${-0.2*scale}"/>
-          <mass value="${back_body_mass}"/>
-          <inertia ixx="0.1" ixy="0.0" ixz="0.0" iyy="1.4" iyz="0.0" izz="1.4"/>
-        </inertial>
-        <buoyancy>
-			<compensation>${back_water_displaced_mass/back_body_mass}</compensation>
-			<origin xyz="${-0.6*scale} 0 ${-0.15*scale}"/>
-			<limit radius="0.1"/>
-			<damping rpy="20 20 20" xyz="20 40 50"/>
-			<windVelocity>${windType}</windVelocity>
-			<frontal_area>0.04</frontal_area>
-			<lateral_area>0.06</lateral_area>
-			<lateral_length>1.2</lateral_length>
-	  		<waterVelocity>${waterType}</waterVelocity>
-        </buoyancy>
-    </link>
-    <joint name="back_r_joint" type="revolute">
-        <parent link="center_r_link"/>
-        <child link="back_r_link"/>
-        <origin rpy="0 0 0" xyz="${-0.5*scale} ${-0.39*scale} 0"/>
-	<limit effort="50" velocity="5" lower="0" upper="0" />
-            <dynamics damping="1.0"/>
-            <axis xyz="1 0 0"/>
-    </joint>
-    <link name="front_r_link">
-    	<visual>
-    	<origin rpy="0 0 0"  xyz="0 0 0"/>
-          <geometry>
-           	<mesh filename="package://usv_sim/meshes/simpleHull3/frontRight.dae" scale="${scale} ${scale} ${scale}"/>
-          </geometry>
-    	</visual>
-        <collision>
-          <origin rpy="0 0 0"  xyz="0 0 0"/>
-          <geometry>
-           	<mesh filename="package://usv_sim/meshes/simpleHull3/frontRight.dae" scale="${scale} ${scale} ${scale}"/>
-          </geometry>
-        </collision>
-        <inertial>
-            <origin rpy="0 0 0" xyz="${0.4*scale} 0 ${-0.1*scale}"/>
-          <mass value="${front_body_mass}"/>
-          <inertia ixx="0.1" ixy="0.0" ixz="0.0" iyy="1.4" iyz="0.0" izz="1.4"/>
-        </inertial>
-        <buoyancy>
-          	<compensation>${front_water_displaced_mass/front_body_mass}</compensation>
-          	<origin xyz="${0.4*scale} 0 ${-0.05*scale}"/>
-          	<limit radius="0.1"/>
-          	<damping rpy="20 20 20" xyz="20 40 50"/>
-          	<windVelocity>${windType}</windVelocity>
-			<frontal_area>0.04</frontal_area>
-			<lateral_area>0.06</lateral_area>
-			<lateral_length>1.2</lateral_length>
-	  		<waterVelocity>${waterType}</waterVelocity>
-        </buoyancy>
-    </link>
-    <joint name="front_r_joint" type="revolute">
-        <parent link="center_r_link"/>
-        <child link="front_r_link"/>
-        <origin rpy="0 0 0" xyz="${1.3*scale} ${-0.2*scale} 0"/>
-	<limit effort="50" velocity="5" lower="0" upper="0" />
-            <dynamics damping="1.0"/>
-            <axis xyz="1 0 0"/>
-    </joint>
+<xacro xmlns:xacro="http://www.ros.org/wiki/xacro" name="right_hull">
+  <!--MR1 BASE LINK-->
+  <link name="center_r_link">
+    <inertial>
+      <origin xyz="${-1.2619*scale} ${-1.71630000002334E-07*scale} ${-0.038115*scale}" rpy="0 0 0" />
+      <mass value="${3.333*scale}" />
+      <inertia ixx="0.61191" ixy="6.46809999999998E-05" ixz="0.0040806" iyy="3.5097" iyz="1.36870000000023E-05" izz="3.5471" />
+    </inertial>
+    <visual>
+      <origin xyz="0 0 0" rpy="1.5707963267949 0 0" />
+      <geometry>
+        <mesh filename="package://usv_sim/meshes/Hull-Middle.STL" />
+      </geometry>
+      <material name="">
+        <color rgba="0.75294 0.75294 0.75294 1" />
+      </material>
+    </visual>
+    <collision>
+      <origin xyz="0 0 0" rpy="1.5707963267949 0 0" />
+      <geometry>
+        <mesh filename="package://usv_sim/meshes/Hull-Middle.STL" />
+      </geometry>
+    </collision>
+    <buoyancy>
+      <compensation>${middle_water_displaced_mass/middle_body_mass}</compensation>
+      <origin xyz="${-1.2619*scale} ${-1.71630000002334E-07*scale} ${-0.038115*scale}" rpy="0 0 0"/>
+      <limit radius="0.1"/>
+      <damping rpy="20 20 20" xyz="20 40 50"/>
+      <windVelocity>${windType}</windVelocity>
+      <frontal_area>0.0</frontal_area>
+      <lateral_area>0.06</lateral_area>
+      <lateral_length>1.2</lateral_length>
+      <waterVelocity>${waterType}</waterVelocity>
+    </buoyancy>
+  </link>
+  <!--MR1 BACK LINK-->
+  <link name="back_r_link">
+    <inertial>
+      <origin xyz="${-0.55395*scale} ${-9.49220000000195E-06*scale} ${-0.031774*scale}" rpy="0 0 0" />
+      <mass value="${3.333*scale}" />
+      <inertia ixx="0.22991" ixy="-2.0064999999998E-05" ixz="-0.032423" iyy="1.3348" iyz="-4.95610000000025E-05" izz="1.2943" />
+    </inertial>
+    <visual>
+      <origin xyz="0 0 0" rpy="1.5707963267949 0 0" />
+      <geometry>
+        <mesh filename="package://usv_sim/meshes/Hull-Back.STL" />
+      </geometry>
+      <material name="">
+        <color rgba="0.75294 0.75294 0.75294 1" />
+      </material>
+    </visual>
+    <collision>
+      <origin xyz="0 0 0" rpy="1.5707963267949 0 0" />
+      <geometry>
+        <mesh filename="package://usv_sim/meshes/Hull-Back.STL" />
+      </geometry>
+    </collision>
+    <buoyancy>
+      <compensation>${back_water_displaced_mass/back_body_mass}</compensation>
+      <origin xyz="${-0.55395*scale} ${-9.49220000000195E-06*scale} ${-0.031774*scale}"/>
+      <limit radius="0.1"/>
+      <damping rpy="20 20 20" xyz="20 40 50"/>
+      <windVelocity>${windType}</windVelocity>
+      <frontal_area>0.04</frontal_area>
+      <lateral_area>0.06</lateral_area>
+      <lateral_length>1.2</lateral_length>
+      <waterVelocity>${waterType}</waterVelocity>
+    </buoyancy>
+  </link>
+  <joint name="back_r_joint" type="revolute">
+    <parent link="center_r_link"/>
+    <child link="back_r_link"/>
+    <origin rpy="0 0 0" xyz="0 0 0"/>
+    <limit effort="50" velocity="5" lower="0" upper="0" />
+    <dynamics damping="1.0"/>
+    <axis xyz="1 0 0"/>
+  </joint>
+  <!--MR1 FRONT LINK-->
+  <link name="front_r_link">
+    <inertial>
+      <origin xyz="${-1.9778*scale} ${4.47239999998292E-07*scale} ${-0.027892*scale}" rpy="0 0 0" />
+      <mass value="${3.333*scale}" />
+      <inertia ixx="0.1729" ixy="1.57389999997978E-07" ixz="0.033027" iyy="1.1311" iyz="3.95489999997434E-07" izz="1.0892" />
+    </inertial>
+    <visual>
+      <origin xyz="0 0 0" rpy="1.5707963267949 0 0" />
+      <geometry>
+        <mesh filename="package://usv_sim/meshes/Hull-Front.STL" />
+      </geometry>
+      <material name="">
+        <color rgba="0.75294 0.75294 0.75294 1" />
+      </material>
+    </visual>
+    <collision>
+      <origin xyz="0 0 0" rpy="1.5707963267949 0 0" />
+      <geometry>
+        <mesh filename="package://usv_sim/meshes/Hull-Front.STL" />
+      </geometry>
+    </collision>
+    <buoyancy>
+      <compensation>${front_water_displaced_mass/front_body_mass}</compensation>
+      <origin xyz="${-1.9778*scale} ${4.47239999998292E-07*scale} ${-0.027892*scale}" rpy="0 0 0" />
+      <limit radius="0.1"/>
+      <damping rpy="20 20 20" xyz="20 40 50"/>
+      <windVelocity>${windType}</windVelocity>
+      <frontal_area>0.04</frontal_area>
+      <lateral_area>0.06</lateral_area>
+      <lateral_length>1.2</lateral_length>
+      <waterVelocity>${waterType}</waterVelocity>
+    </buoyancy>
+  </link>
+  <joint name="front_r_joint" type="revolute">
+    <parent link="center_r_link"/>
+    <child link="front_r_link"/>
+    <origin rpy="0 0 0" xyz="0 0 0"/>
+    <limit effort="50" velocity="5" lower="0" upper="0" />
+    <dynamics damping="1.0"/>
+    <axis xyz="1 0 0"/>
+  </joint>
 </xacro>

Commit message: removed yaw adjustment from buoyancy

File: usv_sim/xacro/mr1_left_hull.xacro (robot description, xacro)
@@ -25,5 +25,5 @@
     <buoyancy>
       <compensation>${middle_water_displaced_mass/middle_body_mass}</compensation>
-      <origin xyz="${-1.2619*scale} ${-1.71630000002334E-07*scale} ${-0.038115*scale}" rpy="0 0 ${-ninety_degrees}"/>
+      <origin xyz="${-1.2619*scale} ${-1.71630000002334E-07*scale} ${-0.038115*scale}" rpy="0 0 0"/>
       <limit radius="0.1"/>
       <damping rpy="20 20 20" xyz="20 40 50"/>
@@ -59,5 +59,5 @@
     <buoyancy>
       <compensation>${back_water_displaced_mass/back_body_mass}</compensation>
-      <origin xyz="${-0.55395*scale} ${-9.49220000000195E-06*scale} ${-0.031774*scale}"rpy="0 0 ${-ninety_degrees}"/>
+      <origin xyz="${-0.55395*scale} ${-9.49220000000195E-06*scale} ${-0.031774*scale}" rpy="0 0 0"/>
       <limit radius="0.1"/>
       <damping rpy="20 20 20" xyz="20 40 50"/>
@@ -101,5 +101,5 @@
     <buoyancy>
       <compensation>${front_water_displaced_mass/front_body_mass}</compensation>
-      <origin xyz="${-1.9778*scale} ${4.47239999998292E-07*scale} ${-0.027892*scale}" rpy="0 0 ${-ninety_degrees}" />
+      <origin xyz="${-1.9778*scale} ${4.47239999998292E-07*scale} ${-0.027892*scale}" rpy="0 0 0" />
       <limit radius="0.1"/>
       <damping rpy="20 20 20" xyz="20 40 50"/>
