Commit message: changed yaw value back to 0 for visual and collision

File: usv_sim/xacro/mr1_left_hull.xacro (robot description, xacro)
@@ -4,10 +4,10 @@
   <link name="base_link">
     <inertial>
-      <origin xyz="${-1.2619*scale} ${-1.71630000002334E-07*scale} ${-0.038115*scale}" rpy="0 0 ${-ninety_degrees}" />
+      <origin xyz="${-1.2619*scale} ${-1.71630000002334E-07*scale} ${-0.038115*scale}" rpy="0 0 0" />
       <mass value="${3.333*scale}" />
       <inertia ixx="0.61191" ixy="6.46809999999998E-05" ixz="0.0040806" iyy="3.5097" iyz="1.36870000000023E-05" izz="3.5471" />
     </inertial>
     <visual>
-      <origin xyz="0 0 0" rpy="1.5707963267949 0 ${-ninety_degrees}" />
+      <origin xyz="0 0 0" rpy="1.5707963267949 0 0" />
       <geometry>
         <mesh filename="package://usv_sim/meshes/Hull-Middle.STL" />
@@ -18,5 +18,5 @@
     </visual>
     <collision>
-      <origin xyz="0 0 0" rpy="1.5707963267949 0 ${-ninety_degrees}" />
+      <origin xyz="0 0 0" rpy="1.5707963267949 0 0" />
       <geometry>
         <mesh filename="package://usv_sim/meshes/Hull-Middle.STL" />
@@ -38,10 +38,10 @@
   <link name="back_l_link">
     <inertial>
-      <origin xyz="${-0.55395*scale} ${-9.49220000000195E-06*scale} ${-0.031774*scale}" rpy="0 0 ${-ninety_degrees}" />
+      <origin xyz="${-0.55395*scale} ${-9.49220000000195E-06*scale} ${-0.031774*scale}" rpy="0 0 0" />
       <mass value="${3.333*scale}" />
       <inertia ixx="0.22991" ixy="-2.0064999999998E-05" ixz="-0.032423" iyy="1.3348" iyz="-4.95610000000025E-05" izz="1.2943" />
     </inertial>
     <visual>
-      <origin xyz="0 0 0" rpy="1.5707963267949 0 ${-ninety_degrees}" />
+      <origin xyz="0 0 0" rpy="1.5707963267949 0 0" />
       <geometry>
         <mesh filename="package://usv_sim/meshes/Hull-Back.STL" />
@@ -52,5 +52,5 @@
     </visual>
     <collision>
-      <origin xyz="0 0 0" rpy="1.5707963267949 0 ${-ninety_degrees}" />
+      <origin xyz="0 0 0" rpy="1.5707963267949 0 0" />
       <geometry>
         <mesh filename="package://usv_sim/meshes/Hull-Back.STL" />
@@ -59,5 +59,5 @@
     <buoyancy>
       <compensation>${back_water_displaced_mass/back_body_mass}</compensation>
-      <origin xyz="${-0.55395*scale} ${-9.49220000000195E-06*scale} ${-0.031774*scale}" rpy="0 0 0"/>
+      <origin xyz="${-0.55395*scale} ${-9.49220000000195E-06*scale} ${-0.031774*scale}"/>
       <limit radius="0.1"/>
       <damping rpy="20 20 20" xyz="20 40 50"/>
@@ -80,10 +80,10 @@
   <link name="front_l_link">
     <inertial>
-      <origin xyz="${-1.9778*scale} ${4.47239999998292E-07*scale} ${-0.027892*scale}" rpy="0 0 ${-ninety_degrees}" />
+      <origin xyz="${-1.9778*scale} ${4.47239999998292E-07*scale} ${-0.027892*scale}" rpy="0 0 0" />
       <mass value="${3.333*scale}" />
       <inertia ixx="0.1729" ixy="1.57389999997978E-07" ixz="0.033027" iyy="1.1311" iyz="3.95489999997434E-07" izz="1.0892" />
     </inertial>
     <visual>
-      <origin xyz="0 0 0" rpy="1.5707963267949 0 ${-ninety_degrees}" />
+      <origin xyz="0 0 0" rpy="1.5707963267949 0 0" />
       <geometry>
         <mesh filename="package://usv_sim/meshes/Hull-Front.STL" />
@@ -94,5 +94,5 @@
     </visual>
     <collision>
-      <origin xyz="0 0 0" rpy="1.5707963267949 0 ${-ninety_degrees}" />
+      <origin xyz="0 0 0" rpy="1.5707963267949 0 0" />
       <geometry>
         <mesh filename="package://usv_sim/meshes/Hull-Front.STL" />

File: usv_sim/xacro/mr1_right_hull.xacro (robot description, xacro)
@@ -4,10 +4,10 @@
   <link name="center_r_link">
     <inertial>
-      <origin xyz="${-1.2619*scale} ${-1.71630000002334E-07*scale} ${-0.038115*scale}" rpy="0 0 ${-ninety_degrees}" />
+      <origin xyz="${-1.2619*scale} ${-1.71630000002334E-07*scale} ${-0.038115*scale}" rpy="0 0 0" />
       <mass value="${3.333*scale}" />
       <inertia ixx="0.61191" ixy="6.46809999999998E-05" ixz="0.0040806" iyy="3.5097" iyz="1.36870000000023E-05" izz="3.5471" />
     </inertial>
     <visual>
-      <origin xyz="0 0 0" rpy="1.5707963267949 0 ${-ninety_degrees}" />
+      <origin xyz="0 0 0" rpy="1.5707963267949 0 0" />
       <geometry>
         <mesh filename="package://usv_sim/meshes/Hull-Middle.STL" />
@@ -18,5 +18,5 @@
     </visual>
     <collision>
-      <origin xyz="0 0 0" rpy="1.5707963267949 0 ${-ninety_degrees}" />
+      <origin xyz="0 0 0" rpy="1.5707963267949 0 0" />
       <geometry>
         <mesh filename="package://usv_sim/meshes/Hull-Middle.STL" />
@@ -38,10 +38,10 @@
   <link name="back_r_link">
     <inertial>
-      <origin xyz="${-0.55395*scale} ${-9.49220000000195E-06*scale} ${-0.031774*scale}" rpy="0 0 ${-ninety_degrees}" />
+      <origin xyz="${-0.55395*scale} ${-9.49220000000195E-06*scale} ${-0.031774*scale}" rpy="0 0 0" />
       <mass value="${3.333*scale}" />
       <inertia ixx="0.22991" ixy="-2.0064999999998E-05" ixz="-0.032423" iyy="1.3348" iyz="-4.95610000000025E-05" izz="1.2943" />
     </inertial>
     <visual>
-      <origin xyz="0 0 0" rpy="1.5707963267949 0 ${-ninety_degrees}" />
+      <origin xyz="0 0 0" rpy="1.5707963267949 0 0" />
       <geometry>
         <mesh filename="package://usv_sim/meshes/Hull-Back.STL" />
@@ -52,5 +52,5 @@
     </visual>
     <collision>
-      <origin xyz="0 0 0" rpy="1.5707963267949 0 ${-ninety_degrees}" />
+      <origin xyz="0 0 0" rpy="1.5707963267949 0 0" />
       <geometry>
         <mesh filename="package://usv_sim/meshes/Hull-Back.STL" />
@@ -59,5 +59,5 @@
     <buoyancy>
       <compensation>${back_water_displaced_mass/back_body_mass}</compensation>
-      <origin xyz="${-0.55395*scale} ${-9.49220000000195E-06*scale} ${-0.031774*scale}" rpy="0 0 0"/>
+      <origin xyz="${-0.55395*scale} ${-9.49220000000195E-06*scale} ${-0.031774*scale}"/>
       <limit radius="0.1"/>
       <damping rpy="20 20 20" xyz="20 40 50"/>
@@ -80,10 +80,10 @@
   <link name="front_r_link">
     <inertial>
-      <origin xyz="${-1.9778*scale} ${4.47239999998292E-07*scale} ${-0.027892*scale}" rpy="0 0 ${-ninety_degrees}" />
+      <origin xyz="${-1.9778*scale} ${4.47239999998292E-07*scale} ${-0.027892*scale}" rpy="0 0 0" />
       <mass value="${3.333*scale}" />
       <inertia ixx="0.1729" ixy="1.57389999997978E-07" ixz="0.033027" iyy="1.1311" iyz="3.95489999997434E-07" izz="1.0892" />
     </inertial>
     <visual>
-      <origin xyz="0 0 0" rpy="1.5707963267949 0 ${-ninety_degrees}" />
+      <origin xyz="0 0 0" rpy="1.5707963267949 0 0" />
       <geometry>
         <mesh filename="package://usv_sim/meshes/Hull-Front.STL" />
@@ -94,5 +94,5 @@
     </visual>
     <collision>
-      <origin xyz="0 0 0" rpy="1.5707963267949 0 ${-ninety_degrees}" />
+      <origin xyz="0 0 0" rpy="1.5707963267949 0 0" />
       <geometry>
         <mesh filename="package://usv_sim/meshes/Hull-Front.STL" />
