Commit message: added necessary variables

File: usv_sim/xacro/mr1.xacro (robot description, xacro)
@@ -1,4 +1,9 @@
 <?xml version="1.0"?>
 <robot xmlns:xacro="http://www.ros.org/wiki/xacro" name="mr1">
+    <xacro:arg name="windType" default="global" />
+    <xacro:arg name="waterType" default="global" />
+    <xacro:property name="windType" value="$(arg windType)" />
+    <xacro:property name="waterType" value="$(arg waterType)" />
+    <xacro:property name="windType" value="global"/>
     <xacro:include filename="$(find usv_sim)/xacro/mr1_base_frame.xacro" />
     <xacro:include filename="$(find usv_sim)/xacro/mr1_hull.xacro" />

Commit message: now imports left and right hull and creates joints

File: usv_sim/xacro/mr1.xacro (robot description, xacro)
@@ -7,6 +7,15 @@
     <xacro:property name="windType" value="global"/>
     <xacro:include filename="$(find usv_sim)/xacro/mr1_base_frame.xacro" />
-    <xacro:include filename="$(find usv_sim)/xacro/mr1_hull.xacro" />
-    <xacro:hull_link name="left_hull" parentLink="left_beam_attachment" />
-    <xacro:hull_link name="right_hull" parentLink="right_beam_attachment" />
+    <xacro:include filename="$(find usv_sim)/xacro/mr1_right_hull.xacro" />
+    <xacro:include filename="$(find usv_sim)/xacro/mr1_left_hull.xacro" />
+    <joint name="right_hull_joint" type="fixed">
+        <parent link="right_beam_attachment"/>
+        <child link="center_r_link" />
+        <origin rpy="0 0 ${ninety_degrees}" xyz="0 0 0"/>
+    </joint>
+    <joint name="left_hull_joint" type="fixed">
+        <parent link="left_beam_attachment"/>
+        <child link="base_link" />
+        <origin rpy="0 0 ${ninety_degrees}" xyz="0 0 0"/>
+    </joint>
 </robot>

Commit message: changed joint x and z origin, frame now attaches to middle of hull

File: usv_sim/xacro/mr1.xacro (robot description, xacro)
@@ -1,4 +1,4 @@
 <?xml version="1.0"?>
-<robot xmlns:xacro="http://www.ros.org/wiki/xacro" name="mr1">
+<robot xmlns:xacro="http://www.ros.org/wiki/xacro" name="sailboat">
     <xacro:arg name="windType" default="global" />
     <xacro:arg name="waterType" default="global" />
@@ -6,16 +6,16 @@
     <xacro:property name="waterType" value="$(arg waterType)" />
     <xacro:property name="windType" value="global"/>
+    <xacro:include filename="$(find usv_sim)/xacro/mr1_left_hull.xacro" />
     <xacro:include filename="$(find usv_sim)/xacro/mr1_base_frame.xacro" />
     <xacro:include filename="$(find usv_sim)/xacro/mr1_right_hull.xacro" />
-    <xacro:include filename="$(find usv_sim)/xacro/mr1_left_hull.xacro" />
     <joint name="right_hull_joint" type="fixed">
         <parent link="right_beam_attachment"/>
         <child link="center_r_link" />
-        <origin rpy="0 0 ${ninety_degrees}" xyz="0 0 0"/>
+        <origin rpy="0 0 ${ninety_degrees}" xyz="${-0.44*scale} 0 ${-0.8*scale}"/>
     </joint>
     <joint name="left_hull_joint" type="fixed">
         <parent link="left_beam_attachment"/>
         <child link="base_link" />
-        <origin rpy="0 0 ${ninety_degrees}" xyz="0 0 0"/>
+        <origin rpy="0 0 ${ninety_degrees}" xyz="${0.44*scale} 0 ${-0.8*scale}"/>
     </joint>
 </robot>

Commit message: moved properties from hulls to here

File: usv_sim/xacro/mr1.xacro (robot description, xacro)
@@ -1,4 +1,17 @@
 <?xml version="1.0"?>
 <robot xmlns:xacro="http://www.ros.org/wiki/xacro" name="sailboat">
+    <xacro:property name="PI" value="3.1415926535897931"/>
+    <!-- Body properties -->
+    <xacro:property name="front_body_mass" value="5"/>
+    <xacro:property name="back_body_mass" value="5"/>
+    <xacro:property name="middle_body_mass" value="5"/>
+    <xacro:property name="rear_body_mass" value="5"/>
+    <xacro:property name="front_body_mass" value="2"/>
+    <xacro:property name="back_water_displaced_mass" value="40"/>
+    <xacro:property name="middle_water_displaced_mass" value="40"/>
+    <xacro:property name="front_water_displaced_mass" value="25"/>
+    <xacro:property name="scale" value="0.3"/>
+    <xacro:property name="bl1" value=".1" />
+    <xacro:property name="bl2" value=".1" />
     <xacro:arg name="windType" default="global" />
     <xacro:arg name="waterType" default="global" />

Commit message: added rudder, moved base frame closer to hulls

File: usv_sim/xacro/mr1.xacro (robot description, xacro)
@@ -22,13 +22,14 @@
     <xacro:include filename="$(find usv_sim)/xacro/mr1_base_frame.xacro" />
     <xacro:include filename="$(find usv_sim)/xacro/mr1_right_hull.xacro" />
+    <xacro:rudder_xacro />
     <joint name="right_hull_joint" type="fixed">
         <parent link="right_beam_attachment"/>
         <child link="center_r_link" />
-        <origin rpy="0 0 ${ninety_degrees}" xyz="${-0.44*scale} 0 ${-0.8*scale}"/>
+        <origin rpy="0 0 ${ninety_degrees}" xyz="${-0.44*scale} 0 ${-0.6*scale}"/>
     </joint>
     <joint name="left_hull_joint" type="fixed">
         <parent link="left_beam_attachment"/>
         <child link="base_link" />
-        <origin rpy="0 0 ${ninety_degrees}" xyz="${0.44*scale} 0 ${-0.8*scale}"/>
+        <origin rpy="0 0 ${ninety_degrees}" xyz="${0.44*scale} 0 ${-0.6*scale}"/>
     </joint>
 </robot>

Commit message: added foil dynamics plugin for sail and rudder

File: usv_sim/xacro/mr1.xacro (robot description, xacro)
@@ -33,3 +33,80 @@
         <origin rpy="0 0 ${ninety_degrees}" xyz="${0.44*scale} 0 ${-0.6*scale}"/>
     </joint>
+   <!-- Defining sail model -->
+    <link name="sail">
+		<inertial>
+		    	<origin rpy="0 0 0" xyz="-0.3 0 0.4"/>
+			<mass value="1" />
+			<inertia
+			  ixx="0.4708"
+			  ixy="0.0"
+			  iyy="0.5208"
+			  ixz="0.0"
+			  iyz="0.0"
+			  izz="0.0508"/>
+		</inertial>
+	    <collision name="collision">
+            <geometry>
+              <mesh filename="package://usv_sim/meshes/simpleHull3/sail.dae" scale="0.5 0.5 0.5"/>
+            </geometry>
+            <origin rpy="0 0 0" xyz="0 0 0"/>
+	    </collision>
+	    <visual name="visual">
+            <geometry>
+              <mesh filename="package://usv_sim/meshes/simpleHull3/sail.dae" scale="0.5 0.5 0.5"/>
+            </geometry>
+            <origin rpy="0 0 0" xyz="0 0 0"/>
+	    </visual>
+    </link>
+    <joint name="sail_joint" type="revolute">
+        <parent link="base_cube"/>
+        <child link="sail"/>
+        <origin rpy="0 0 0" xyz="0 0 ${scale*0.2}"/>
+        <dynamics damping="1.0"/>
+        <axis xyz="0 0 1"/>
+        <limit effort="100" velocity="70" lower="-${PI}" upper="${PI}" />
+    </joint>
+        <!-- Plugin list -->
+    <gazebo>
+	<plugin name="usv_sail_plugin" filename="libfoil_dynamics_plugin.so">
+	  <link_type>sail</link_type>
+	  <a0>0</a0>
+	  <cla>3.0</cla>
+	  <cda>3.0</cda>
+	  <cma>-1.8</cma>
+	  <alpha_stall>0.785</alpha_stall>
+	  <cla_stall>-3.85</cla_stall>
+	  <cda_stall>-0.9233984055</cda_stall>
+	  <cma_stall>0</cma_stall>
+	  <cp>0 0 0</cp>
+	  <joint_name>sail_joint</joint_name>
+	  <area>1.44</area>
+	  <fluid_density>1.2041</fluid_density>
+	  <forward>-1 0 0</forward>
+	  <upward>0 1 0</upward>
+	  <link_name>sail</link_name>
+	  <fluidVelocity>${windType}</fluidVelocity>
+      </plugin>
+      <plugin name="usv_sail_plugin" filename="libfoil_dynamics_plugin.so">
+	<link_type>rudder</link_type>
+	<a0>0</a0>
+	<cla>0.8</cla>
+	<cda>0.3</cda>
+	<alpha_stall>0.785</alpha_stall>
+	<cla_stall>-0.85</cla_stall>
+	<cda_stall>-0.3233984055</cda_stall>
+	<cp>0 0 0</cp>
+	<area>1</area>
+	<fluid_density>1000</fluid_density>
+	<forward>1 0 0</forward>
+	<upward>0 1 0</upward>
+	<link_name>rudder</link_name>
+	<fluidVelocity>${waterType}</fluidVelocity>
+      </plugin>
+      <plugin name="freefloating_gazebo_control" filename="libfreefloating_gazebo_control.so">
+        <switchService>switch</switchService>
+        <updateRate>100</updateRate>
+        <link>base_link</link>
+      </plugin>
+    </gazebo>
 </robot>

Commit message: added keel, added fluid plugin for keel and rudder

File: usv_sim/xacro/mr1.xacro (robot description, xacro)
@@ -62,8 +62,40 @@
         <parent link="base_cube"/>
         <child link="sail"/>
-        <origin rpy="0 0 0" xyz="0 0 ${scale*0.2}"/>
+        <origin rpy="0 0 ${ninety_degrees}" xyz="0 0 ${scale*0.2}"/>
         <dynamics damping="1.0"/>
         <axis xyz="0 0 1"/>
         <limit effort="100" velocity="70" lower="-${PI}" upper="${PI}" />
+    </joint>
+    <link name="keel">
+        <inertial>
+            <mass value="30" />
+            <inertia
+            ixx="0.4708"
+            ixy="0.0"
+            iyy="0.5208"
+            ixz="0.0"
+            iyz="0.0"
+            izz="0.0508"/>
+        </inertial>
+        <collision name="collision">
+            <geometry>
+                <box size="0.12 0.02 0.5" />
+            </geometry>
+            <origin rpy="0 0 0" xyz="0 0 0"/>
+        </collision>
+        <visual name="visual">
+            <geometry>
+                <mesh filename="package://usv_sim/meshes/simpleHull3/box.dae" scale="0.12 0.02 0.5"/>
+            </geometry>
+            <origin rpy="0 0 0" xyz="0 0 0"/>
+        </visual>
+    </link>
+    <joint name="keel_joint" type="revolute">
+        <parent link="base_cube"/>
+        <child link="keel"/>
+        <origin rpy="0 0 ${ninety_degrees}" xyz="0 0 -0.35"/>
+        <dynamics damping="1.0"/>
+        <axis xyz="0 0 1"/>
+        <limit effort="30" velocity="5" lower="0" upper="0" />
     </joint>
         <!-- Plugin list -->
@@ -88,20 +120,37 @@
 	  <fluidVelocity>${windType}</fluidVelocity>
       </plugin>
-      <plugin name="usv_sail_plugin" filename="libfoil_dynamics_plugin.so">
-	<link_type>rudder</link_type>
-	<a0>0</a0>
-	<cla>0.8</cla>
-	<cda>0.3</cda>
-	<alpha_stall>0.785</alpha_stall>
-	<cla_stall>-0.85</cla_stall>
-	<cda_stall>-0.3233984055</cda_stall>
-	<cp>0 0 0</cp>
-	<area>1</area>
-	<fluid_density>1000</fluid_density>
-	<forward>1 0 0</forward>
-	<upward>0 1 0</upward>
-	<link_name>rudder</link_name>
-	<fluidVelocity>${waterType}</fluidVelocity>
-      </plugin>
+    <plugin name="usv_sail_plugin" filename="libfoil_dynamics_plugin.so">
+        <link_type>rudder</link_type>
+        <a0>0</a0>
+        <cla>0.8</cla>
+        <cda>0.3</cda>
+        <alpha_stall>0.785</alpha_stall>
+        <cla_stall>-0.85</cla_stall>
+        <cda_stall>-0.3233984055</cda_stall>
+        <cp>0 0 0</cp>
+        <area>1</area>
+        <fluid_density>1000</fluid_density>
+        <forward>1 0 0</forward>
+        <upward>0 1 0</upward>
+        <link_name>rudder</link_name>
+        <fluidVelocity>${waterType}</fluidVelocity>
+    </plugin>
+    <plugin name="usv_sail_plugin" filename="libusv_sailing_plugin.so">
+		  <link_type>keel</link_type>
+		  <a0>0</a0>
+		  <cla>10.0</cla>
+		  <cda>8.0</cda>
+		  <alpha_stall>0.785</alpha_stall>
+		  <cla_stall>-10.0</cla_stall>
+		  <cda_stall>-5.0</cda_stall>
+		  <cp>0 0 0</cp>
+		  <area>1.0</area>
+		  <fluid_density>1000</fluid_density>
+		  <forward>1 0 0</forward>
+		  <upward>0 1 0</upward>
+            <limit effort="100" velocity="70" lower="-${PI}" upper="${PI}" />
+	  <link_name>keel</link_name>
+		  <fluidVelocity>${waterType}</fluidVelocity>
+    </plugin>
       <plugin name="freefloating_gazebo_control" filename="libfreefloating_gazebo_control.so">
         <switchService>switch</switchService>

Commit message: changed scale to 1, modified hull join to work for new hull, reformated

File: usv_sim/xacro/mr1.xacro (robot description, xacro)
@@ -11,5 +11,5 @@
     <xacro:property name="middle_water_displaced_mass" value="40"/>
     <xacro:property name="front_water_displaced_mass" value="25"/>
-    <xacro:property name="scale" value="0.3"/>
+    <xacro:property name="scale" value="1"/>
     <xacro:property name="bl1" value=".1" />
     <xacro:property name="bl2" value=".1" />
@@ -26,36 +26,30 @@
         <parent link="right_beam_attachment"/>
         <child link="center_r_link" />
-        <origin rpy="0 0 ${ninety_degrees}" xyz="${-0.44*scale} 0 ${-0.6*scale}"/>
+        <origin rpy="0 0 ${ninety_degrees}" xyz="0 ${1.2*scale} ${-beam_to_hull_length}"/>
     </joint>
     <joint name="left_hull_joint" type="fixed">
         <parent link="left_beam_attachment"/>
         <child link="base_link" />
-        <origin rpy="0 0 ${ninety_degrees}" xyz="${0.44*scale} 0 ${-0.6*scale}"/>
+        <origin rpy="0 0 ${ninety_degrees}" xyz="0 ${1.2*scale} ${-beam_to_hull_length}"/>
     </joint>
-   <!-- Defining sail model -->
+    <!-- Defining sail model -->
     <link name="sail">
-		<inertial>
-		    	<origin rpy="0 0 0" xyz="-0.3 0 0.4"/>
-			<mass value="1" />
-			<inertia
-			  ixx="0.4708"
-			  ixy="0.0"
-			  iyy="0.5208"
-			  ixz="0.0"
-			  iyz="0.0"
-			  izz="0.0508"/>
-		</inertial>
-	    <collision name="collision">
+        <inertial>
+            <origin rpy="0 0 0" xyz="-0.3 0 0.4"/>
+            <mass value="1" />
+            <inertia ixx="0.4708" ixy="0.0" iyy="0.5208" ixz="0.0" iyz="0.0" izz="0.0508"/>
+        </inertial>
+        <collision name="collision">
             <geometry>
-              <mesh filename="package://usv_sim/meshes/simpleHull3/sail.dae" scale="0.5 0.5 0.5"/>
+                <mesh filename="package://usv_sim/meshes/simpleHull3/sail.dae" scale="0.5 0.5 0.5"/>
             </geometry>
             <origin rpy="0 0 0" xyz="0 0 0"/>
-	    </collision>
-	    <visual name="visual">
+        </collision>
+        <visual name="visual">
             <geometry>
-              <mesh filename="package://usv_sim/meshes/simpleHull3/sail.dae" scale="0.5 0.5 0.5"/>
+                <mesh filename="package://usv_sim/meshes/simpleHull3/sail.dae" scale="0.5 0.5 0.5"/>
             </geometry>
             <origin rpy="0 0 0" xyz="0 0 0"/>
-	    </visual>
+        </visual>
     </link>
     <joint name="sail_joint" type="revolute">
@@ -70,11 +64,5 @@
         <inertial>
             <mass value="30" />
-            <inertia
-            ixx="0.4708"
-            ixy="0.0"
-            iyy="0.5208"
-            ixz="0.0"
-            iyz="0.0"
-            izz="0.0508"/>
+            <inertia ixx="0.4708" ixy="0.0" iyy="0.5208" ixz="0.0" iyz="0.0" izz="0.0508"/>
         </inertial>
         <collision name="collision">
@@ -94,68 +82,68 @@
         <parent link="base_cube"/>
         <child link="keel"/>
-        <origin rpy="0 0 ${ninety_degrees}" xyz="0 0 -0.35"/>
+        <origin rpy="0 0 ${ninety_degrees}" xyz="0 0 ${-0.6*scale}"/>
         <dynamics damping="1.0"/>
         <axis xyz="0 0 1"/>
         <limit effort="30" velocity="5" lower="0" upper="0" />
     </joint>
-        <!-- Plugin list -->
+    <!-- Plugin list -->
     <gazebo>
-	<plugin name="usv_sail_plugin" filename="libfoil_dynamics_plugin.so">
-	  <link_type>sail</link_type>
-	  <a0>0</a0>
-	  <cla>3.0</cla>
-	  <cda>3.0</cda>
-	  <cma>-1.8</cma>
-	  <alpha_stall>0.785</alpha_stall>
-	  <cla_stall>-3.85</cla_stall>
-	  <cda_stall>-0.9233984055</cda_stall>
-	  <cma_stall>0</cma_stall>
-	  <cp>0 0 0</cp>
-	  <joint_name>sail_joint</joint_name>
-	  <area>1.44</area>
-	  <fluid_density>1.2041</fluid_density>
-	  <forward>-1 0 0</forward>
-	  <upward>0 1 0</upward>
-	  <link_name>sail</link_name>
-	  <fluidVelocity>${windType}</fluidVelocity>
-      </plugin>
-    <plugin name="usv_sail_plugin" filename="libfoil_dynamics_plugin.so">
-        <link_type>rudder</link_type>
-        <a0>0</a0>
-        <cla>0.8</cla>
-        <cda>0.3</cda>
-        <alpha_stall>0.785</alpha_stall>
-        <cla_stall>-0.85</cla_stall>
-        <cda_stall>-0.3233984055</cda_stall>
-        <cp>0 0 0</cp>
-        <area>1</area>
-        <fluid_density>1000</fluid_density>
-        <forward>1 0 0</forward>
-        <upward>0 1 0</upward>
-        <link_name>rudder</link_name>
-        <fluidVelocity>${waterType}</fluidVelocity>
-    </plugin>
-    <plugin name="usv_sail_plugin" filename="libusv_sailing_plugin.so">
-		  <link_type>keel</link_type>
-		  <a0>0</a0>
-		  <cla>10.0</cla>
-		  <cda>8.0</cda>
-		  <alpha_stall>0.785</alpha_stall>
-		  <cla_stall>-10.0</cla_stall>
-		  <cda_stall>-5.0</cda_stall>
-		  <cp>0 0 0</cp>
-		  <area>1.0</area>
-		  <fluid_density>1000</fluid_density>
-		  <forward>1 0 0</forward>
-		  <upward>0 1 0</upward>
+        <plugin name="usv_sail_plugin" filename="libfoil_dynamics_plugin.so">
+            <link_type>sail</link_type>
+            <a0>0</a0>
+            <cla>3.0</cla>
+            <cda>3.0</cda>
+            <cma>-1.8</cma>
+            <alpha_stall>0.785</alpha_stall>
+            <cla_stall>-3.85</cla_stall>
+            <cda_stall>-0.9233984055</cda_stall>
+            <cma_stall>0</cma_stall>
+            <cp>0 0 0</cp>
+            <joint_name>sail_joint</joint_name>
+            <area>1.44</area>
+            <fluid_density>1.2041</fluid_density>
+            <forward>-1 0 0</forward>
+            <upward>0 1 0</upward>
+            <link_name>sail</link_name>
+            <fluidVelocity>${windType}</fluidVelocity>
+        </plugin>
+        <plugin name="usv_sail_plugin" filename="libfoil_dynamics_plugin.so">
+            <link_type>rudder</link_type>
+            <a0>0</a0>
+            <cla>0.8</cla>
+            <cda>0.3</cda>
+            <alpha_stall>0.785</alpha_stall>
+            <cla_stall>-0.85</cla_stall>
+            <cda_stall>-0.3233984055</cda_stall>
+            <cp>0 0 0</cp>
+            <area>1</area>
+            <fluid_density>1000</fluid_density>
+            <forward>1 0 0</forward>
+            <upward>0 1 0</upward>
+            <link_name>rudder</link_name>
+            <fluidVelocity>${waterType}</fluidVelocity>
+        </plugin>
+        <plugin name="usv_sail_plugin" filename="libfoil_dynamics_plugin.so">
+            <link_type>keel</link_type>
+            <a0>0</a0>
+            <cla>10.0</cla>
+            <cda>8.0</cda>
+            <alpha_stall>0.785</alpha_stall>
+            <cla_stall>-10.0</cla_stall>
+            <cda_stall>-5.0</cda_stall>
+            <cp>0 0 0</cp>
+            <area>1.0</area>
+            <fluid_density>1000</fluid_density>
+            <forward>1 0 0</forward>
+            <upward>0 1 0</upward>
             <limit effort="100" velocity="70" lower="-${PI}" upper="${PI}" />
-	  <link_name>keel</link_name>
-		  <fluidVelocity>${waterType}</fluidVelocity>
-    </plugin>
-      <plugin name="freefloating_gazebo_control" filename="libfreefloating_gazebo_control.so">
-        <switchService>switch</switchService>
-        <updateRate>100</updateRate>
-        <link>base_link</link>
-      </plugin>
+            <link_name>keel</link_name>
+            <fluidVelocity>${waterType}</fluidVelocity>
+        </plugin>
+        <plugin name="freefloating_gazebo_control" filename="libfreefloating_gazebo_control.so">
+            <switchService>switch</switchService>
+            <updateRate>100</updateRate>
+            <link>base_link</link>
+        </plugin>
     </gazebo>
 </robot>
