Commit message: changed yaw by -90 degrees

File: usv_sim/xacro/mr1.xacro (robot description, xacro)
@@ -19,6 +19,6 @@
     <xacro:property name="waterType" value="$(arg waterType)" />
     <xacro:property name="windType" value="global"/>
+    <xacro:include filename="$(find usv_sim)/xacro/mr1_base_frame.xacro" />
     <xacro:include filename="$(find usv_sim)/xacro/mr1_left_hull.xacro" />
-    <xacro:include filename="$(find usv_sim)/xacro/mr1_base_frame.xacro" />
     <xacro:include filename="$(find usv_sim)/xacro/mr1_right_hull.xacro" />
     <xacro:rudder_xacro />
@@ -26,10 +26,10 @@
         <parent link="right_beam_attachment"/>
         <child link="center_r_link" />
-        <origin rpy="0 0 ${ninety_degrees}" xyz="0 ${1.2*scale} ${-beam_to_hull_length}"/>
+        <origin rpy="0 0 ${ninety_degrees}" xyz="${1.2*scale} 0 ${-beam_to_hull_length}"/>
     </joint>
     <joint name="left_hull_joint" type="fixed">
         <parent link="left_beam_attachment"/>
         <child link="base_link" />
-        <origin rpy="0 0 ${ninety_degrees}" xyz="0 ${1.2*scale} ${-beam_to_hull_length}"/>
+        <origin rpy="0 0 ${ninety_degrees}" xyz="${1.2*scale} 0 ${-beam_to_hull_length}"/>
     </joint>
     <!-- Defining sail model -->
@@ -56,5 +56,5 @@
         <parent link="base_cube"/>
         <child link="sail"/>
-        <origin rpy="0 0 ${ninety_degrees}" xyz="0 0 ${scale*0.2}"/>
+        <origin rpy="0 0 0" xyz="0 0 ${scale*0.2}"/>
         <dynamics damping="1.0"/>
         <axis xyz="0 0 1"/>
@@ -82,5 +82,5 @@
         <parent link="base_cube"/>
         <child link="keel"/>
-        <origin rpy="0 0 ${ninety_degrees}" xyz="0 0 ${-0.6*scale}"/>
+        <origin rpy="0 0 0" xyz="0 0 ${-0.6*scale}"/>
         <dynamics damping="1.0"/>
         <axis xyz="0 0 1"/>

File: usv_sim/xacro/mr1_base_frame.xacro (robot description, xacro)
@@ -11,5 +11,5 @@
         <box size="${base_cube_length} ${base_cube_length} ${base_cube_length}"/>
       </geometry>
-      <origin rpy="0 0 0" xyz="0 0 0"/>
+      <origin rpy="0 0 ${-ninety_degrees}" xyz="0 0 0"/>
     </visual>
     <collision>
@@ -17,5 +17,5 @@
         <box size="${base_cube_length} ${base_cube_length} ${base_cube_length}"/>
       </geometry>
-      <origin rpy="0 0 0" xyz="0 0 0"/>
+      <origin rpy="0 0 ${-ninety_degrees}" xyz="0 0 0"/>
     </collision>
     <inertial>
@@ -29,11 +29,11 @@
         <cylinder radius="${beam_radius}" length="${beam_length}"/>
       </geometry>
-      <origin rpy="${ninety_degrees} 0 0" xyz="0 0 0"/>
-    </visual>
-    <collision>
-      <geometry>
-        <cylinder radius="${beam_radius}" length="${beam_length}"/>
-      </geometry>
-      <origin rpy="${ninety_degrees} 0 0" xyz="0 0 0"/>
+      <origin rpy="${ninety_degrees} 0 ${-ninety_degrees}" xyz="0 0 0"/>
+    </visual>
+    <collision>
+      <geometry>
+        <cylinder radius="${beam_radius}" length="${beam_length}"/>
+      </geometry>
+      <origin rpy="${ninety_degrees} 0 ${-ninety_degrees}" xyz="0 0 0"/>
     </collision>
     <inertial>
@@ -45,5 +45,5 @@
     <parent link="base_cube"/>
     <child link="rear_beam"/>
-    <origin xyz="0 ${-(beam_length/2)+(base_cube_length/2)} 0"/>
+    <origin xyz="${-(beam_length/2)+(base_cube_length/2)} 0 0"/>
   </joint>
   <link name="right_beam">
@@ -53,5 +53,5 @@
       </geometry>
       <!-- rotate beam 90 degrees -->
-      <origin rpy="0 ${ninety_degrees} 0" xyz="0 0 0"/>
+      <origin rpy="0 ${ninety_degrees} ${-ninety_degrees}" xyz="0 0 0"/>
     </visual>
     <collision>
@@ -60,5 +60,5 @@
       </geometry>
       <!-- rotate beam 90 degrees -->
-      <origin rpy="0 ${ninety_degrees} 0" xyz="0 0 0"/>
+      <origin rpy="0 ${ninety_degrees} ${-ninety_degrees}" xyz="0 0 0"/>
     </collision>
     <inertial>
@@ -70,5 +70,5 @@
     <parent link="base_cube"/>
     <child link="right_beam"/>
-    <origin xyz="${(beam_length/2)+(base_cube_length/2)} 0 0"/>
+    <origin xyz="0 ${(beam_length/2)+(base_cube_length/2)} 0"/>
   </joint>
   <link name="left_beam">
@@ -77,11 +77,11 @@
         <cylinder radius="${beam_radius}" length="${beam_length}"/>
       </geometry>
-      <origin rpy="0 ${ninety_degrees} 0" xyz="0 0 0"/>
-    </visual>
-    <collision>
-      <geometry>
-        <cylinder radius="${beam_radius}" length="${beam_length}"/>
-      </geometry>
-      <origin rpy="0 ${ninety_degrees} 0" xyz="0 0 0"/>
+      <origin rpy="0 ${ninety_degrees} ${-ninety_degrees}" xyz="0 0 0"/>
+    </visual>
+    <collision>
+      <geometry>
+        <cylinder radius="${beam_radius}" length="${beam_length}"/>
+      </geometry>
+      <origin rpy="0 ${ninety_degrees} ${-ninety_degrees}" xyz="0 0 0"/>
     </collision>
     <inertial>
@@ -93,5 +93,5 @@
     <parent link="base_cube"/>
     <child link="left_beam"/>
-    <origin xyz="${-((beam_length/2)+(base_cube_length/2))} 0 0"/>
+    <origin xyz="0 ${-((beam_length/2)+(base_cube_length/2))} 0"/>
   </joint>
  <link name="left_beam_attachment">
@@ -101,12 +101,12 @@
       </geometry>
       <!--origin z offset = length/2 -->
-      <origin rpy="0 0 0" xyz="0 0 ${-beam_to_hull_length/2}"/>
-    </visual>
-    <collision>
-      <geometry>
-        <cylinder radius="${beam_radius}" length="${beam_to_hull_length}"/>
-      </geometry>
-      <!--origin z offset = length/2 -->
-      <origin rpy="0 0 0" xyz="0 0 ${-beam_to_hull_length/2}"/>
+      <origin rpy="0 0 ${-ninety_degrees}" xyz="0 0 ${-beam_to_hull_length/2}"/>
+    </visual>
+    <collision>
+      <geometry>
+        <cylinder radius="${beam_radius}" length="${beam_to_hull_length}"/>
+      </geometry>
+      <!--origin z offset = length/2 -->
+      <origin rpy="0 0 ${-ninety_degrees}" xyz="0 0 ${-beam_to_hull_length/2}"/>
     </collision>
     <inertial>
@@ -119,5 +119,5 @@
     <child link="left_beam_attachment"/>
     <!--origin x offset = beam_length/2 -radius -->
-    <origin xyz="-0.25 0 0"/>
+    <origin xyz="0 -0.25 0"/>
   </joint>
  <link name="right_beam_attachment">
@@ -127,12 +127,12 @@
       </geometry>
       <!--origin z offset = length/2 -->
-      <origin rpy="0 0 0" xyz="0 0 ${-beam_to_hull_length/2}"/>
-    </visual>
-    <collision>
-      <geometry>
-        <cylinder radius="${beam_radius}" length="${beam_to_hull_length}"/>
-      </geometry>
-      <!--origin z offset = length/2 -->
-      <origin rpy="0 0 0" xyz="0 0 ${-beam_to_hull_length/2}"/>
+      <origin rpy="0 0 ${-ninety_degrees}" xyz="0 0 ${-beam_to_hull_length/2}"/>
+    </visual>
+    <collision>
+      <geometry>
+        <cylinder radius="${beam_radius}" length="${beam_to_hull_length}"/>
+      </geometry>
+      <!--origin z offset = length/2 -->
+      <origin rpy="0 0 ${-ninety_degrees}" xyz="0 0 ${-beam_to_hull_length/2}"/>
     </collision>
     <inertial>
@@ -145,5 +145,5 @@
     <child link="right_beam_attachment"/>
     <!--origin x offset = beam_length/2 -radius -->
-    <origin xyz="0.25 0 0"/>
+    <origin xyz="0 0.25 0"/>
   </joint>
  <link name="rudder_attachment">
@@ -153,12 +153,12 @@
       </geometry>
       <!--origin z offset = length/2 -->
-      <origin rpy="0 0 0" xyz="0 0 ${-beam_to_hull_length/2}"/>
-    </visual>
-    <collision>
-      <geometry>
-        <cylinder radius="${beam_radius}" length="${beam_to_hull_length}"/>
-      </geometry>
-      <!--origin z offset = length/2 -->
-      <origin rpy="0 0 0" xyz="0 0 ${-beam_to_hull_length/2}"/>
+      <origin rpy="0 0 ${-ninety_degrees}" xyz="0 0 ${-beam_to_hull_length/2}"/>
+    </visual>
+    <collision>
+      <geometry>
+        <cylinder radius="${beam_radius}" length="${beam_to_hull_length}"/>
+      </geometry>
+      <!--origin z offset = length/2 -->
+      <origin rpy="0 0 ${-ninety_degrees}" xyz="0 0 ${-beam_to_hull_length/2}"/>
     </collision>
     <inertial>
@@ -171,5 +171,5 @@
     <child link="rudder_attachment"/>
     <!--origin x offset = beam_length/2 -radius -->
-    <origin xyz="0 -0.25 0"/>
+    <origin xyz="-0.25 0 0"/>
   </joint>
   <!-- Rudder link -->
@@ -202,5 +202,5 @@
             <parent link="rudder_attachment"/>
             <child link="rudder"/>
-            <origin rpy="0 0 ${ninety_degrees}" xyz="0 0 ${-0.6*scale}"/>
+            <origin rpy="0 0 0" xyz="0 0 ${-0.6*scale}"/>
 <!--            <origin rpy="0 0 ${ninety_degrees" xyz="0 0 ${-0.6*scale}"/-->
             <dynamics damping="1.0"/>

File: usv_sim/xacro/mr1_left_hull.xacro (robot description, xacro)
@@ -4,10 +4,10 @@
   <link name="base_link">
     <inertial>
-      <origin xyz="${-1.2619*scale} ${-1.71630000002334E-07*scale} ${-0.038115*scale}" rpy="0 0 0" />
+      <origin xyz="${-1.2619*scale} ${-1.71630000002334E-07*scale} ${-0.038115*scale}" rpy="0 0 ${-ninety_degrees}" />
       <mass value="${3.333*scale}" />
       <inertia ixx="0.61191" ixy="6.46809999999998E-05" ixz="0.0040806" iyy="3.5097" iyz="1.36870000000023E-05" izz="3.5471" />
     </inertial>
     <visual>
-      <origin xyz="0 0 0" rpy="1.5707963267949 0 0" />
+      <origin xyz="0 0 0" rpy="1.5707963267949 0 ${-ninety_degrees}" />
       <geometry>
         <mesh filename="package://usv_sim/meshes/Hull-Middle.STL" />
@@ -18,5 +18,5 @@
     </visual>
     <collision>
-      <origin xyz="0 0 0" rpy="1.5707963267949 0 0" />
+      <origin xyz="0 0 0" rpy="1.5707963267949 0 ${-ninety_degrees}" />
       <geometry>
         <mesh filename="package://usv_sim/meshes/Hull-Middle.STL" />
@@ -25,5 +25,5 @@
     <buoyancy>
       <compensation>${middle_water_displaced_mass/middle_body_mass}</compensation>
-      <origin xyz="${-1.2619*scale} ${-1.71630000002334E-07*scale} ${-0.038115*scale}" rpy="0 0 0"/>
+      <origin xyz="${-1.2619*scale} ${-1.71630000002334E-07*scale} ${-0.038115*scale}" rpy="0 0 ${-ninety_degrees}"/>
       <limit radius="0.1"/>
       <damping rpy="20 20 20" xyz="20 40 50"/>
@@ -38,10 +38,10 @@
   <link name="back_l_link">
     <inertial>
-      <origin xyz="${-0.55395*scale} ${-9.49220000000195E-06*scale} ${-0.031774*scale}" rpy="0 0 0" />
+      <origin xyz="${-0.55395*scale} ${-9.49220000000195E-06*scale} ${-0.031774*scale}" rpy="0 0 ${-ninety_degrees}" />
       <mass value="${3.333*scale}" />
       <inertia ixx="0.22991" ixy="-2.0064999999998E-05" ixz="-0.032423" iyy="1.3348" iyz="-4.95610000000025E-05" izz="1.2943" />
     </inertial>
     <visual>
-      <origin xyz="0 0 0" rpy="1.5707963267949 0 0" />
+      <origin xyz="0 0 0" rpy="1.5707963267949 0 ${-ninety_degrees}" />
       <geometry>
         <mesh filename="package://usv_sim/meshes/Hull-Back.STL" />
@@ -52,5 +52,5 @@
     </visual>
     <collision>
-      <origin xyz="0 0 0" rpy="1.5707963267949 0 0" />
+      <origin xyz="0 0 0" rpy="1.5707963267949 0 ${-ninety_degrees}" />
       <geometry>
         <mesh filename="package://usv_sim/meshes/Hull-Back.STL" />
@@ -59,5 +59,5 @@
     <buoyancy>
       <compensation>${back_water_displaced_mass/back_body_mass}</compensation>
-      <origin xyz="${-0.55395*scale} ${-9.49220000000195E-06*scale} ${-0.031774*scale}"/>
+      <origin xyz="${-0.55395*scale} ${-9.49220000000195E-06*scale} ${-0.031774*scale}"rpy="0 0 ${-ninety_degrees}"/>
       <limit radius="0.1"/>
       <damping rpy="20 20 20" xyz="20 40 50"/>
@@ -80,10 +80,10 @@
   <link name="front_l_link">
     <inertial>
-      <origin xyz="${-1.9778*scale} ${4.47239999998292E-07*scale} ${-0.027892*scale}" rpy="0 0 0" />
+      <origin xyz="${-1.9778*scale} ${4.47239999998292E-07*scale} ${-0.027892*scale}" rpy="0 0 ${-ninety_degrees}" />
       <mass value="${3.333*scale}" />
       <inertia ixx="0.1729" ixy="1.57389999997978E-07" ixz="0.033027" iyy="1.1311" iyz="3.95489999997434E-07" izz="1.0892" />
     </inertial>
     <visual>
-      <origin xyz="0 0 0" rpy="1.5707963267949 0 0" />
+      <origin xyz="0 0 0" rpy="1.5707963267949 0 ${-ninety_degrees}" />
       <geometry>
         <mesh filename="package://usv_sim/meshes/Hull-Front.STL" />
@@ -94,5 +94,5 @@
     </visual>
     <collision>
-      <origin xyz="0 0 0" rpy="1.5707963267949 0 0" />
+      <origin xyz="0 0 0" rpy="1.5707963267949 0 ${-ninety_degrees}" />
       <geometry>
         <mesh filename="package://usv_sim/meshes/Hull-Front.STL" />
@@ -101,5 +101,5 @@
     <buoyancy>
       <compensation>${front_water_displaced_mass/front_body_mass}</compensation>
-      <origin xyz="${-1.9778*scale} ${4.47239999998292E-07*scale} ${-0.027892*scale}" rpy="0 0 0" />
+      <origin xyz="${-1.9778*scale} ${4.47239999998292E-07*scale} ${-0.027892*scale}" rpy="0 0 ${-ninety_degrees}" />
       <limit radius="0.1"/>
       <damping rpy="20 20 20" xyz="20 40 50"/>

File: usv_sim/xacro/mr1_right_hull.xacro (robot description, xacro)
@@ -4,10 +4,10 @@
   <link name="center_r_link">
     <inertial>
-      <origin xyz="${-1.2619*scale} ${-1.71630000002334E-07*scale} ${-0.038115*scale}" rpy="0 0 0" />
+      <origin xyz="${-1.2619*scale} ${-1.71630000002334E-07*scale} ${-0.038115*scale}" rpy="0 0 ${-ninety_degrees}" />
       <mass value="${3.333*scale}" />
       <inertia ixx="0.61191" ixy="6.46809999999998E-05" ixz="0.0040806" iyy="3.5097" iyz="1.36870000000023E-05" izz="3.5471" />
     </inertial>
     <visual>
-      <origin xyz="0 0 0" rpy="1.5707963267949 0 0" />
+      <origin xyz="0 0 0" rpy="1.5707963267949 0 ${-ninety_degrees}" />
       <geometry>
         <mesh filename="package://usv_sim/meshes/Hull-Middle.STL" />
@@ -18,5 +18,5 @@
     </visual>
     <collision>
-      <origin xyz="0 0 0" rpy="1.5707963267949 0 0" />
+      <origin xyz="0 0 0" rpy="1.5707963267949 0 ${-ninety_degrees}" />
       <geometry>
         <mesh filename="package://usv_sim/meshes/Hull-Middle.STL" />
@@ -25,5 +25,5 @@
     <buoyancy>
       <compensation>${middle_water_displaced_mass/middle_body_mass}</compensation>
-      <origin xyz="${-1.2619*scale} ${-1.71630000002334E-07*scale} ${-0.038115*scale}" rpy="0 0 0"/>
+      <origin xyz="${-1.2619*scale} ${-1.71630000002334E-07*scale} ${-0.038115*scale}" rpy="0 0 ${-ninety_degrees}"/>
       <limit radius="0.1"/>
       <damping rpy="20 20 20" xyz="20 40 50"/>
@@ -38,10 +38,10 @@
   <link name="back_r_link">
     <inertial>
-      <origin xyz="${-0.55395*scale} ${-9.49220000000195E-06*scale} ${-0.031774*scale}" rpy="0 0 0" />
+      <origin xyz="${-0.55395*scale} ${-9.49220000000195E-06*scale} ${-0.031774*scale}" rpy="0 0 ${-ninety_degrees}" />
       <mass value="${3.333*scale}" />
       <inertia ixx="0.22991" ixy="-2.0064999999998E-05" ixz="-0.032423" iyy="1.3348" iyz="-4.95610000000025E-05" izz="1.2943" />
     </inertial>
     <visual>
-      <origin xyz="0 0 0" rpy="1.5707963267949 0 0" />
+      <origin xyz="0 0 0" rpy="1.5707963267949 0 ${-ninety_degrees}" />
       <geometry>
         <mesh filename="package://usv_sim/meshes/Hull-Back.STL" />
@@ -52,5 +52,5 @@
     </visual>
     <collision>
-      <origin xyz="0 0 0" rpy="1.5707963267949 0 0" />
+      <origin xyz="0 0 0" rpy="1.5707963267949 0 ${-ninety_degrees}" />
       <geometry>
         <mesh filename="package://usv_sim/meshes/Hull-Back.STL" />
@@ -59,5 +59,5 @@
     <buoyancy>
       <compensation>${back_water_displaced_mass/back_body_mass}</compensation>
-      <origin xyz="${-0.55395*scale} ${-9.49220000000195E-06*scale} ${-0.031774*scale}"/>
+      <origin xyz="${-0.55395*scale} ${-9.49220000000195E-06*scale} ${-0.031774*scale}" rpy="0 0 ${-ninety_degrees}"/>
       <limit radius="0.1"/>
       <damping rpy="20 20 20" xyz="20 40 50"/>
@@ -80,10 +80,10 @@
   <link name="front_r_link">
     <inertial>
-      <origin xyz="${-1.9778*scale} ${4.47239999998292E-07*scale} ${-0.027892*scale}" rpy="0 0 0" />
+      <origin xyz="${-1.9778*scale} ${4.47239999998292E-07*scale} ${-0.027892*scale}" rpy="0 0 ${-ninety_degrees}" />
       <mass value="${3.333*scale}" />
       <inertia ixx="0.1729" ixy="1.57389999997978E-07" ixz="0.033027" iyy="1.1311" iyz="3.95489999997434E-07" izz="1.0892" />
     </inertial>
     <visual>
-      <origin xyz="0 0 0" rpy="1.5707963267949 0 0" />
+      <origin xyz="0 0 0" rpy="1.5707963267949 0 ${-ninety_degrees}" />
       <geometry>
         <mesh filename="package://usv_sim/meshes/Hull-Front.STL" />
@@ -94,5 +94,5 @@
     </visual>
     <collision>
-      <origin xyz="0 0 0" rpy="1.5707963267949 0 0" />
+      <origin xyz="0 0 0" rpy="1.5707963267949 0 ${-ninety_degrees}" />
       <geometry>
         <mesh filename="package://usv_sim/meshes/Hull-Front.STL" />
@@ -101,5 +101,5 @@
     <buoyancy>
       <compensation>${front_water_displaced_mass/front_body_mass}</compensation>
-      <origin xyz="${-1.9778*scale} ${4.47239999998292E-07*scale} ${-0.027892*scale}" rpy="0 0 0" />
+      <origin xyz="${-1.9778*scale} ${4.47239999998292E-07*scale} ${-0.027892*scale}" rpy="0 0 ${-ninety_degrees}" />
       <limit radius="0.1"/>
       <damping rpy="20 20 20" xyz="20 40 50"/>

Commit message: rotate hull join 180 degrees instead of 90

File: usv_sim/xacro/mr1.xacro (robot description, xacro)
@@ -26,10 +26,10 @@
         <parent link="right_beam_attachment"/>
         <child link="center_r_link" />
-        <origin rpy="0 0 ${ninety_degrees}" xyz="${1.2*scale} 0 ${-beam_to_hull_length}"/>
+        <origin rpy="0 0 ${PI}" xyz="${-1.2*scale} 0 ${-beam_to_hull_length}"/>
     </joint>
     <joint name="left_hull_joint" type="fixed">
         <parent link="left_beam_attachment"/>
         <child link="base_link" />
-        <origin rpy="0 0 ${ninety_degrees}" xyz="${1.2*scale} 0 ${-beam_to_hull_length}"/>
+        <origin rpy="0 0 ${PI}" xyz="${-1.2*scale} 0 ${-beam_to_hull_length}"/>
     </joint>
     <!-- Defining sail model -->

Commit message: replaced sail with mr1 sail

File: usv_sim/xacro/mr1.xacro (robot description, xacro)
@@ -36,27 +36,30 @@
     <link name="sail">
         <inertial>
-            <origin rpy="0 0 0" xyz="-0.3 0 0.4"/>
-            <mass value="1" />
-            <inertia ixx="0.4708" ixy="0.0" iyy="0.5208" ixz="0.0" iyz="0.0" izz="0.0508"/>
+            <origin xyz="0.90666 0.1166 -1.75660000000071E-05" rpy="0 0 0" />
+            <mass value="5.1671" />
+            <inertia ixx="0.1332" ixy="-0.12422" ixz="0.000254509999999992" iyy="1.4044" iyz="-1.91999999999932E-05" izz="1.5154" />
         </inertial>
-        <collision name="collision">
+        <visual>
+            <origin xyz="0 0 0" rpy="1.5707963267949 0 0" />
             <geometry>
-                <mesh filename="package://usv_sim/meshes/simpleHull3/sail.dae" scale="0.5 0.5 0.5"/>
+                <mesh filename="package://usv_sim/meshes/sail.STL" />
             </geometry>
-            <origin rpy="0 0 0" xyz="0 0 0"/>
+            <material name="">
+                <color rgba="0.49804 0.49804 0.49804 1" />
+            </material>
+        </visual>
+        <collision>
+            <origin xyz="0 0 0" rpy="1.5707963267949 0 0" />
+            <geometry>
+                <mesh filename="package://usv_sim/meshes/sail.STL" />
+            </geometry>
         </collision>
-        <visual name="visual">
-            <geometry>
-                <mesh filename="package://usv_sim/meshes/simpleHull3/sail.dae" scale="0.5 0.5 0.5"/>
-            </geometry>
-            <origin rpy="0 0 0" xyz="0 0 0"/>
-        </visual>
     </link>
     <joint name="sail_joint" type="revolute">
         <parent link="base_cube"/>
         <child link="sail"/>
-        <origin rpy="0 0 0" xyz="0 0 ${scale*0.2}"/>
+        <origin rpy="${-ninety_degrees} ${-ninety_degrees} ${PI}" xyz="0 0 ${scale*0.05}"/>
         <dynamics damping="1.0"/>
-        <axis xyz="0 0 1"/>
+        <axis xyz="1 0 0"/>
         <limit effort="100" velocity="70" lower="-${PI}" upper="${PI}" />
     </joint>
